Commit message: Fix Gazebo DOF Bot mesh visibility

File: ros2_ws/src/tactile_sim/urdf/dofbot_gazebo.urdf.xacro (robot description, xacro)
@@ -1,5 +1,5 @@
 <?xml version="1.0"?>
 <robot name="yahboom_dofbot" xmlns:xacro="http://www.ros.org/wiki/xacro">
-  <xacro:property name="mesh_root" value="package://tactile_sim/meshes"/>
+  <xacro:property name="mesh_root" value="file://$(find tactile_sim)/meshes"/>
   <link name="world"/>
   <joint name="world_to_base" type="fixed">

Commit message: Add MoveIt Gazebo demo and simulated wrist sensors

File: ros2_ws/src/tactile_sim/urdf/dofbot_gazebo.urdf.xacro (robot description, xacro)
@@ -24,7 +24,13 @@
     </visual>
     <collision>
-      <origin xyz="0 0 0" rpy="0 0 0"/>
-      <geometry>
-        <mesh filename="${mesh_root}/base_link.STL"/>
+      <origin xyz="0 -0.07 0.002" rpy="0 0 0"/>
+      <geometry>
+        <box size="0.12 0.26 0.004"/>
+      </geometry>
+    </collision>
+    <collision>
+      <origin xyz="0 -0.005 0.0435" rpy="0 0 0"/>
+      <geometry>
+        <box size="0.082 0.13 0.079"/>
       </geometry>
     </collision>
@@ -46,7 +52,7 @@
     </visual>
     <collision>
-      <origin xyz="0 0 0" rpy="0 0 0"/>
-      <geometry>
-        <mesh filename="${mesh_root}/link1.STL"/>
+      <origin xyz="0 0 0.026" rpy="0 0 0"/>
+      <geometry>
+        <cylinder radius="0.028" length="0.055"/>
       </geometry>
     </collision>
@@ -76,7 +82,13 @@
     </visual>
     <collision>
-      <origin xyz="0 0 0" rpy="-1.5708 0 1.5708"/>
-      <geometry>
-        <mesh filename="${mesh_root}/link2.STL"/>
+      <origin xyz="0 -0.0665 0" rpy="-1.5708 0 1.5708"/>
+      <geometry>
+        <box size="0.053 0.021 0.045"/>
+      </geometry>
+    </collision>
+    <collision>
+      <origin xyz="0 -0.0135 0.003" rpy="-1.5708 0 1.5708"/>
+      <geometry>
+        <box size="0.055 0.029 0.042"/>
       </geometry>
     </collision>
@@ -106,7 +118,13 @@
     </visual>
     <collision>
-      <origin xyz="0 0 0" rpy="-1.5708 0 1.5708"/>
-      <geometry>
-        <mesh filename="${mesh_root}/link3.STL"/>
+      <origin xyz="0.0006 -0.0665 0" rpy="-1.5708 0 1.5708"/>
+      <geometry>
+        <box size="0.053 0.021 0.045"/>
+      </geometry>
+    </collision>
+    <collision>
+      <origin xyz="0.0006 -0.0135 0.003" rpy="-1.5708 0 1.5708"/>
+      <geometry>
+        <box size="0.055 0.029 0.042"/>
       </geometry>
     </collision>
@@ -136,7 +154,13 @@
     </visual>
     <collision>
-      <origin xyz="0 0 0" rpy="-1.5708 0 1.5708"/>
-      <geometry>
-        <mesh filename="${mesh_root}/link4.STL"/>
+      <origin xyz="0.0011 -0.054 0.016" rpy="-1.5708 0 1.5708"/>
+      <geometry>
+        <box size="0.046 0.097 0.035"/>
+      </geometry>
+    </collision>
+    <collision>
+      <origin xyz="0.0011 -0.0085 0.0035" rpy="-1.5708 0 1.5708"/>
+      <geometry>
+        <box size="0.045 0.029 0.035"/>
       </geometry>
     </collision>
@@ -166,7 +190,19 @@
     </visual>
     <collision>
-      <origin xyz="0 0 0" rpy="0 0 0"/>
-      <geometry>
-        <mesh filename="${mesh_root}/arm_link5.STL"/>
+      <origin xyz="0.0015 0 -0.092" rpy="0 0 0"/>
+      <geometry>
+        <box size="0.023 0.020 0.020"/>
+      </geometry>
+    </collision>
+    <collision>
+      <origin xyz="0.0025 -0.0025 -0.070" rpy="0 0 0"/>
+      <geometry>
+        <box size="0.031 0.055 0.024"/>
+      </geometry>
+    </collision>
+    <collision>
+      <origin xyz="0.03 -0.0055 -0.068" rpy="0 0 0"/>
+      <geometry>
+        <box size="0.024 0.045 0.020"/>
       </geometry>
     </collision>
@@ -196,7 +232,7 @@
     </visual>
     <collision>
-      <origin xyz="0 0 0" rpy="0 0 0"/>
-      <geometry>
-        <mesh filename="${mesh_root}/rlink1.STL"/>
+      <origin xyz="0.0101 0.0014 0.00035" rpy="0 0 0"/>
+      <geometry>
+        <box size="0.048 0.025 0.005"/>
       </geometry>
     </collision>
@@ -226,7 +262,7 @@
     </visual>
     <collision>
-      <origin xyz="0 0 0" rpy="0 0 0"/>
-      <geometry>
-        <mesh filename="${mesh_root}/rlink2.STL"/>
+      <origin xyz="0.0233 0.0046 -0.003" rpy="0 0 0"/>
+      <geometry>
+        <box size="0.054 0.017 0.014"/>
       </geometry>
     </collision>
@@ -255,7 +291,7 @@
     </visual>
     <collision>
-      <origin xyz="0 0 0" rpy="0 0 0"/>
-      <geometry>
-        <mesh filename="${mesh_root}/rlink3.STL"/>
+      <origin xyz="0.015 0 -0.004" rpy="0 0 0"/>
+      <geometry>
+        <box size="0.036 0.006 0.016"/>
       </geometry>
     </collision>
@@ -284,7 +320,7 @@
     </visual>
     <collision>
-      <origin xyz="0 0 0" rpy="0 0 0"/>
-      <geometry>
-        <mesh filename="${mesh_root}/llink1.STL"/>
+      <origin xyz="0.0101 -0.0014 0.001" rpy="0 0 0"/>
+      <geometry>
+        <box size="0.048 0.025 0.005"/>
       </geometry>
     </collision>
@@ -313,7 +349,7 @@
     </visual>
     <collision>
-      <origin xyz="0 0 0" rpy="0 0 0"/>
-      <geometry>
-        <mesh filename="${mesh_root}/llink2.STL"/>
+      <origin xyz="0.0233 -0.0046 -0.003" rpy="0 0 0"/>
+      <geometry>
+        <box size="0.054 0.017 0.014"/>
       </geometry>
     </collision>
@@ -342,7 +378,7 @@
     </visual>
     <collision>
-      <origin xyz="0 0 0" rpy="0 0 0"/>
-      <geometry>
-        <mesh filename="${mesh_root}/llink3.STL"/>
+      <origin xyz="0.015 0 -0.004" rpy="0 0 0"/>
+      <geometry>
+        <box size="0.036 0.006 0.016"/>
       </geometry>
     </collision>
@@ -355,4 +391,245 @@
     <mimic joint="grip_joint" multiplier="-1"/>
   </joint>
+  <link name="ee_link"/>
+  <joint name="arm_tool0_joint" type="fixed">
+    <origin xyz="0 0 -0.105" rpy="0 0 0"/>
+    <parent link="arm_link5"/>
+    <child link="ee_link"/>
+  </joint>
+  <link name="camera_link">
+    <inertial>
+      <origin xyz="0 0 0" rpy="0 0 0"/>
+      <mass value="0.08"/>
+      <inertia ixx="8.0e-05" ixy="0" ixz="0" iyy="2.0e-04" iyz="0" izz="2.0e-04"/>
+    </inertial>
+    <visual>
+      <origin xyz="0 0 0" rpy="0 0 0"/>
+      <geometry>
+        <box size="0.020 0.095 0.030"/>
+      </geometry>
+      <material name="camera_body_light">
+        <color rgba="0.78 0.78 0.80 1"/>
+      </material>
+    </visual>
+    <visual>
+      <origin xyz="0 0.0475 0" rpy="0 1.5708 0"/>
+      <geometry>
+        <cylinder length="0.020" radius="0.015"/>
+      </geometry>
+      <material name="camera_body_light">
+        <color rgba="0.78 0.78 0.80 1"/>
+      </material>
+    </visual>
+    <visual>
+      <origin xyz="0 -0.0475 0" rpy="0 1.5708 0"/>
+      <geometry>
+        <cylinder length="0.020" radius="0.015"/>
+      </geometry>
+      <material name="camera_body_light">
+        <color rgba="0.78 0.78 0.80 1"/>
+      </material>
+    </visual>
+    <visual>
+      <origin xyz="0.013 0 0" rpy="0 0 0"/>
+      <geometry>
+        <box size="0.006 0.095 0.026"/>
+      </geometry>
+      <material name="camera_body_light">
+        <color rgba="0.78 0.78 0.80 1"/>
+      </material>
+    </visual>
+    <visual>
+      <origin xyz="0.013 0.0475 0" rpy="0 1.5708 0"/>
+      <geometry>
+        <cylinder length="0.006" radius="0.013"/>
+      </geometry>
+      <material name="camera_body_light">
+        <color rgba="0.78 0.78 0.80 1"/>
+      </material>
+    </visual>
+    <visual>
+      <origin xyz="0.013 -0.0475 0" rpy="0 1.5708 0"/>
+      <geometry>
+        <cylinder length="0.006" radius="0.013"/>
+      </geometry>
+      <material name="camera_body_light">
+        <color rgba="0.78 0.78 0.80 1"/>
+      </material>
+    </visual>
+    <visual>
+      <origin xyz="-0.013 0 0" rpy="0 0 0"/>
+      <geometry>
+        <box size="0.006 0.095 0.026"/>
+      </geometry>
+      <material name="camera_body_light">
+        <color rgba="0.78 0.78 0.80 1"/>
+      </material>
+    </visual>
+    <visual>
+      <origin xyz="-0.013 0.0475 0" rpy="0 1.5708 0"/>
+      <geometry>
+        <cylinder length="0.006" radius="0.013"/>
+      </geometry>
+      <material name="camera_body_light">
+        <color rgba="0.78 0.78 0.80 1"/>
+      </material>
+    </visual>
+    <visual>
+      <origin xyz="-0.013 -0.0475 0" rpy="0 1.5708 0"/>
+      <geometry>
+        <cylinder length="0.006" radius="0.013"/>
+      </geometry>
+      <material name="camera_body_light">
+        <color rgba="0.78 0.78 0.80 1"/>
+      </material>
+    </visual>
+    <visual>
+      <origin xyz="0.013 0 0" rpy="0 0 0"/>
+      <geometry>
+        <box size="0.004 0.095 0.026"/>
+      </geometry>
+      <material name="camera_front_dark">
+        <color rgba="0.10 0.10 0.10 1"/>
+      </material>
+    </visual>
+    <visual>
+      <origin xyz="0.013 0.0475 0" rpy="0 1.5708 0"/>
+      <geometry>
+        <cylinder length="0.004" radius="0.013"/>
+      </geometry>
+      <material name="camera_front_dark">
+        <color rgba="0.10 0.10 0.10 1"/>
+      </material>
+    </visual>
+    <visual>
+      <origin xyz="0.013 -0.0475 0" rpy="0 1.5708 0"/>
+      <geometry>
+        <cylinder length="0.004" radius="0.013"/>
+      </geometry>
+      <material name="camera_front_dark">
+        <color rgba="0.10 0.10 0.10 1"/>
+      </material>
+    </visual>
+    <collision>
+      <origin xyz="0 0 0" rpy="0 0 0"/>
+      <geometry>
+        <box size="0.032 0.125 0.030"/>
+      </geometry>
+    </collision>
+  </link>
+  <joint name="camera_joint" type="fixed">
+    <origin xyz="0.001 -0.060 0.050" rpy="0 0 -1.5708"/>
+    <parent link="arm_link4"/>
+    <child link="camera_link"/>
+  </joint>
+  <gazebo reference="camera_joint">
+    <preserveFixedJoint>true</preserveFixedJoint>
+  </gazebo>
+  <link name="camera_color_frame"/>
+  <joint name="camera_color_frame_joint" type="fixed">
+    <origin xyz="0 0 0" rpy="0 0 0"/>
+    <parent link="camera_link"/>
+    <child link="camera_color_frame"/>
+  </joint>
+  <link name="camera_color_optical_frame"/>
+  <joint name="camera_color_optical_joint" type="fixed">
+    <origin xyz="0 0 0" rpy="-1.5708 0 -1.5708"/>
+    <parent link="camera_color_frame"/>
+    <child link="camera_color_optical_frame"/>
+  </joint>
+  <link name="camera_depth_frame"/>
+  <joint name="camera_depth_frame_joint" type="fixed">
+    <origin xyz="0 0 0" rpy="0 0 0"/>
+    <parent link="camera_link"/>
+    <child link="camera_depth_frame"/>
+  </joint>
+  <link name="camera_depth_optical_frame"/>
+  <joint name="camera_depth_optical_joint" type="fixed">
+    <origin xyz="0 0 0" rpy="-1.5708 0 -1.5708"/>
+    <parent link="camera_depth_frame"/>
+    <child link="camera_depth_optical_frame"/>
+  </joint>
+  <link name="camera_imu_frame"/>
+  <joint name="camera_imu_frame_joint" type="fixed">
+    <origin xyz="0 0 0" rpy="0 0 0"/>
+    <parent link="camera_link"/>
+    <child link="camera_imu_frame"/>
+  </joint>
+  <link name="camera_imu_optical_frame"/>
+  <joint name="camera_imu_optical_joint" type="fixed">
+    <origin xyz="0 0 0" rpy="-1.5708 0 -1.5708"/>
+    <parent link="camera_imu_frame"/>
+    <child link="camera_imu_optical_frame"/>
+  </joint>
+  <link name="camera_gyro_frame"/>
+  <joint name="camera_gyro_frame_joint" type="fixed">
+    <origin xyz="0 0 0" rpy="0 0 0"/>
+    <parent link="camera_imu_frame"/>
+    <child link="camera_gyro_frame"/>
+  </joint>
+  <link name="camera_gyro_optical_frame"/>
+  <joint name="camera_gyro_optical_joint" type="fixed">
+    <origin xyz="0 0 0" rpy="-1.5708 0 -1.5708"/>
+    <parent link="camera_gyro_frame"/>
+    <child link="camera_gyro_optical_frame"/>
+  </joint>
+  <link name="camera_accel_frame"/>
+  <joint name="camera_accel_frame_joint" type="fixed">
+    <origin xyz="0 0 0" rpy="0 0 0"/>
+    <parent link="camera_imu_frame"/>
+    <child link="camera_accel_frame"/>
+  </joint>
+  <link name="camera_accel_optical_frame"/>
+  <joint name="camera_accel_optical_joint" type="fixed">
+    <origin xyz="0 0 0" rpy="-1.5708 0 -1.5708"/>
+    <parent link="camera_accel_frame"/>
+    <child link="camera_accel_optical_frame"/>
+  </joint>
+  <gazebo reference="camera_link">
+    <sensor name="wrist_rgb_camera" type="camera">
+      <always_on>1</always_on>
+      <update_rate>30</update_rate>
+      <visualize>true</visualize>
+      <topic>camera</topic>
+      <camera>
+        <horizontal_fov>1.204</horizontal_fov>
+        <image>
+          <width>640</width>
+          <height>480</height>
+          <format>R8G8B8</format>
+        </image>
+        <clip>
+          <near>0.03</near>
+          <far>10.0</far>
+        </clip>
+      </camera>
+    </sensor>
+    <sensor name="wrist_depth_camera" type="depth_camera">
+      <always_on>1</always_on>
+      <update_rate>30</update_rate>
+      <visualize>false</visualize>
+      <topic>camera_depth</topic>
+      <camera>
+        <horizontal_fov>1.204</horizontal_fov>
+        <image>
+          <width>640</width>
+          <height>480</height>
+          <format>R_FLOAT32</format>
+        </image>
+        <clip>
+          <near>0.03</near>
+          <far>10.0</far>
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
Commit message: Refactor sim stack for modular grasp pipeline

File: ros2_ws/src/tactile_sim/urdf/dofbot_gazebo.urdf.xacro (robot description, xacro)
@@ -6,5 +6,5 @@
     <parent link="world"/>
     <child link="base_link"/>
-    <origin xyz="0 0 0" rpy="0 0 0"/>
+    <origin xyz="0 0 0" rpy="0 0 -1.57079632679"/>
   </joint>
   <link name="base_link">
@@ -59,9 +59,9 @@
   </link>
   <joint name="arm_joint1" type="revolute">
-    <origin xyz="0 0 0.06605" rpy="-0.010805 0 1.5"/>
+    <origin xyz="0 0 0.06605" rpy="-0.010805 0 4.64159265359"/>
     <parent link="base_link"/>
     <child link="arm_link1"/>
     <axis xyz="0 0 1"/>
-    <limit effort="30" velocity="1.0" lower="-1.5708" upper="1.5708"/>
+    <limit effort="30" velocity="1.0" lower="-3.14159" upper="3.14159"/>
     <dynamics damping="0.2" friction="0.05"/>
   </joint>
@@ -99,5 +99,5 @@
     <child link="arm_link2"/>
     <axis xyz="1 0 0"/>
-    <limit lower="-1.5708" upper="1.5708" effort="100" velocity="1"/>
+    <limit lower="-1.745329" upper="0.0" effort="100" velocity="1"/>
     <dynamics damping="0.2" friction="0.05"/>
   </joint>
@@ -135,5 +135,5 @@
     <child link="arm_link3"/>
     <axis xyz="1 0 0"/>
-    <limit lower="-1.5708" upper="1.5708" effort="100" velocity="1"/>
+    <limit lower="-0.785398" upper="2.094395" effort="100" velocity="1"/>
     <dynamics damping="0.2" friction="0.05"/>
   </joint>
@@ -171,5 +171,5 @@
     <child link="arm_link4"/>
     <axis xyz="1 0 0"/>
-    <limit lower="-1.5708" upper="1.5708" effort="100" velocity="1"/>
+    <limit lower="-0.785398" upper="2.094395" effort="100" velocity="1"/>
     <dynamics damping="0.2" friction="0.05"/>
   </joint>
@@ -638,30 +638,42 @@
     <joint name="arm_joint1">
       <command_interface name="position"/>
-      <state_interface name="position"/>
+      <state_interface name="position">
+        <param name="initial_value">-1.518436</param>
+      </state_interface>
       <state_interface name="velocity"/>
     </joint>
     <joint name="arm_joint2">
       <command_interface name="position"/>
-      <state_interface name="position"/>
+      <state_interface name="position">
+        <param name="initial_value">-1.256637</param>
+      </state_interface>
       <state_interface name="velocity"/>
     </joint>
     <joint name="arm_joint3">
       <command_interface name="position"/>
-      <state_interface name="position"/>
+      <state_interface name="position">
+        <param name="initial_value">1.553343</param>
+      </state_interface>
       <state_interface name="velocity"/>
     </joint>
     <joint name="arm_joint4">
       <command_interface name="position"/>
-      <state_interface name="position"/>
+      <state_interface name="position">
+        <param name="initial_value">1.553343</param>
+      </state_interface>
       <state_interface name="velocity"/>
     </joint>
     <joint name="arm_joint5">
       <command_interface name="position"/>
-      <state_interface name="position"/>
+      <state_interface name="position">
+        <param name="initial_value">-1.570796</param>
+      </state_interface>
       <state_interface name="velocity"/>
     </joint>
     <joint name="grip_joint">
       <command_interface name="position"/>
-      <state_interface name="position"/>
+      <state_interface name="position">
+        <param name="initial_value">0.0</param>
+      </state_interface>
       <state_interface name="velocity"/>
     </joint>

Commit message: Fix sim world alignment and improve web grasp flow

File: ros2_ws/src/tactile_sim/urdf/dofbot_gazebo.urdf.xacro (robot description, xacro)
@@ -2,9 +2,14 @@
 <robot name="yahboom_dofbot" xmlns:xacro="http://www.ros.org/wiki/xacro">
   <xacro:property name="mesh_root" value="file://$(find tactile_sim)/meshes"/>
+  <xacro:arg name="base_world_x" default="0.0"/>
+  <xacro:arg name="base_world_y" default="0.0"/>
+  <xacro:arg name="base_world_z" default="0.0"/>
   <link name="world"/>
   <joint name="world_to_base" type="fixed">
     <parent link="world"/>
     <child link="base_link"/>
-    <origin xyz="0 0 0" rpy="0 0 -1.57079632679"/>
+    <origin
+      xyz="$(arg base_world_x) $(arg base_world_y) $(arg base_world_z)"
+      rpy="0 0 -1.57079632679"/>
   </joint>
   <link name="base_link">
